Commit message: add joint

File: catkin_ws/src/omnibot/urdf/robot.xacro (robot description, xacro)
@@ -1,12 +1,23 @@
 <?xml version="1.0" encoding="UTF-8" ?>
-<robot name="mock_robot" xmlns:xacro="http://www.ros.org/wiki/xacro">
-  <!-- The robot link description -->
+<robot name="mock_robot"
+  xmlns:xacro="http://www.ros.org/wiki/xacro">
   <link name="base_link">
-      <visual>
+    <visual>
       <geometry>
-        <cylinder length="0.3" radius="0.2"/>
-        <origin xyz="0 0 0.15"/>
+        <cylinder length="0.1" radius="0.21"/>
       </geometry>
     </visual>
   </link>
+  <link name="electronic">
+    <visual>
+      <geometry>
+        <cylinder length="0.08" radius="0.1"/>
+      </geometry>
+    </visual>
+  </link>
+  <joint name="electronic_to_base" type="fixed">
+    <parent link="base_link"/>
+    <child link="electronic"/>
+    <origin xyz="0 0 0.05"/>
+  </joint>
 </robot>

Commit message: fix rumus odometry

File: catkin_ws/src/omnibot/urdf/robot.xacro (robot description, xacro)
@@ -4,4 +4,5 @@
   <link name="base_link">
     <visual>
+    <origin xyz="0 0 0.05"/>
       <geometry>
         <cylinder length="0.1" radius="0.21"/>
@@ -19,5 +20,5 @@
     <parent link="base_link"/>
     <child link="electronic"/>
-    <origin xyz="0 0 0.05"/>
+    <origin xyz="0 0 0.1"/>
   </joint>
 </robot>
